File: KiCAD Schematic/original version/BME280 schematic-original-v2.kicad_sch (KiCad schematic)
At the start: 16 parts, among them J1 Conn_01x04, Q1 BSS138, Q2 BSS138, U1 MIC5219-3.3YM5, U2 BME280

Commit message: Update BME280 schematic-original-v2.kicad_sch
Connections:
- net +3.3V: no longer 0.1uF1.2, 4.7uF1.2, C1.1, C2.2, C3.2, J1.GND (Pin_3), JP1.3 (B), R3.2, U1.2 (GND), U2.1 (GND), U2.7 (GND)
- new net GND: 0.1uF1.2, 4.7uF1.2, C1.1, C2.2, C3.2, J1.GND (Pin_3), JP1.3 (B), R3.2, U1.2 (GND), U2.1 (GND), U2.7 (GND)
